File: Hardware/hymTracker/hymTracker.sch (KiCad schematic (older format))
At the start: 16 parts

Commit message: sema cizildi
Parts:
- added J1: DB9_Female, symbol Connector:DB9_Female
- added U1: MP1584_DCDC, symbol mylibs:MP1584_DCDC
- added U2: GY-NEO6MV2, symbol Adem:GY-NEO6MV2
- gave numbers to parts that had none: 16
Connections:
- net labels added: ANALOG_SENSOR1, ANALOG_SENSOR2, DIGITAL_GIRIS, I2C_SCL, I2C_SDA, MIKROFON, VCC
- net labels removed: Cikis
- wire segments 44 -> 64
- no-connect marks 2 -> 13
Other:
- note added: "5V'a ayarlanacak"
- moved on the sheet: A1, C1, C2, D1, Q1, R1, R10, R2, R3, R4, R5, R6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

Commit message: pcb ye hazir
Parts:
- C1: footprint (none) -> Capacitor_SMD:C_0805_2012Metric
- C2: footprint (none) -> Capacitor_SMD:C_1206_3216Metric
- D1: footprint (none) -> LED_SMD:LED_0805_2012Metric
- J1: footprint (none) -> Connector_Dsub:DSUB-9_Female_Horizontal_P2.77x2.84mm_EdgePinOffset7.70mm_Housed_MountingHolesOffset9.12mm
- R1, R10, R2, R3, R4, R5, R6, R7, R8, R9: footprint (none) -> Resistor_SMD:R_0805_2012Metric
- RV1: footprint (none) -> Potentiometer_THT:Potentiometer_ACP_CA9-V10_Vertical_Hole
- U1: footprint (none) -> hymTracker:MP1854EN_board
- U2: footprint (none) -> hymTracker:Neo6
Changed lines of the file:
@@
 F 0 "R4" V 3945 2015 50  0000 C CNN
 F 1 "8K8" V 4000 2205 50  0000 C CNN
-F 2 "" V 3930 2200 50  0001 C CNN
+F 2 "Resistor_SMD:R_0805_2012Metric" V 3930 2200 50  0001 C CNN
 F 3 "~" H 4000 2200 50  0001 C CNN
 	1    4000 2200
@@
 F 0 "R5" V 3950 2115 50  0000 C CNN
 F 1 "3K3" V 4000 2300 50  0000 C CNN
-F 2 "" V 3930 2300 50  0001 C CNN
+F 2 "Resistor_SMD:R_0805_2012Metric" V 3930 2300 50  0001 C CNN
 F 3 "~" H 4000 2300 50  0001 C CNN
 	1    4000 2300
@@
 F 0 "R6" V 3950 2215 50  0000 C CNN
 F 1 "2K2" V 4000 2395 50  0000 C CNN
-F 2 "" V 3930 2400 50  0001 C CNN
+F 2 "Resistor_SMD:R_0805_2012Metric" V 3930 2400 50  0001 C CNN
 F 3 "~" H 4000 2400 50  0001 C CNN
 	1    4000 2400
@@
 P 4300 2800
 F 0 "R9" H 4230 2754 50  0000 R CNN
-F 1 "270" H 4230 2845 50  0000 R CNN
-F 2 "" V 4230 2800 50  0001 C CNN
+F 1 "270" V 4300 2850 50  0000 R CNN
+F 2 "Resistor_SMD:R_0805_2012Metric" V 4230 2800 50  0001 C CNN
 F 3 "~" H 4300 2800 50  0001 C CNN
 	1    4300 2800
@@
 F 0 "R3" V 4040 2180 50  0000 C CNN
 F 1 "220" V 3995 2000 50  0000 C CNN
-F 2 "" V 3930 2000 50  0001 C CNN
+F 2 "Resistor_SMD:R_0805_2012Metric" V 3930 2000 50  0001 C CNN
 F 3 "~" H 4000 2000 50  0001 C CNN
 	1    4000 2000
@@
 F 0 "D1" H 4410 1905 50  0000 C CNN
 F 1 "LED" H 4395 2085 50  0000 C CNN
-F 2 "" H 4400 2000 50  0001 C CNN
+F 2 "LED_SMD:LED_0805_2012Metric" H 4400 2000 50  0001 C CNN
 F 3 "~" H 4400 2000 50  0001 C CNN
 	1    4400 2000
@@
 F 0 "C1" H 4715 2846 50  0000 L CNN
 F 1 "100n" H 4715 2755 50  0000 L CNN
-F 2 "" H 4638 2650 50  0001 C CNN
+F 2 "Capacitor_SMD:C_0805_2012Metric" H 4638 2650 50  0001 C CNN
 F 3 "~" H 4600 2800 50  0001 C CNN
 	1    4600 2800
@@
 F 0 "C2" V 5035 2400 50  0000 C CNN
 F 1 "4u7" V 4755 2400 50  0000 C CNN
-F 2 "" H 4938 2250 50  0001 C CNN
+F 2 "Capacitor_SMD:C_1206_3216Metric" H 4938 2250 50  0001 C CNN
 F 3 "~" H 4900 2400 50  0001 C CNN
 	1    4900 2400
@@
 F 0 "RV1" H 5240 2354 50  0000 R CNN
 F 1 "100K" H 5240 2445 50  0000 R CNN
-F 2 "" H 5300 2400 50  0001 C CNN
+F 2 "Potentiometer_THT:Potentiometer_ACP_CA9-V10_Vertical_Hole" H 5300 2400 50  0001 C CNN
 F 3 "~" H 5300 2400 50  0001 C CNN
 	1    5300 2400
@@
 P 5300 2800
 F 0 "R10" H 5230 2754 50  0000 R CNN
-F 1 "100K" H 5230 2845 50  0000 R CNN
-F 2 "" V 5230 2800 50  0001 C CNN
+F 1 "100K" V 5300 2900 50  0000 R CNN
+F 2 "Resistor_SMD:R_0805_2012Metric" V 5230 2800 50  0001 C CNN
 F 3 "~" H 5300 2800 50  0001 C CNN
 	1    5300 2800
@@
 F 0 "R8" V 4457 4050 50  0000 C CNN
 F 1 "10K" V 4366 4050 50  0000 C CNN
-F 2 "" V 4180 4050 50  0001 C CNN
+F 2 "Resistor_SMD:R_0805_2012Metric" V 4180 4050 50  0001 C CNN
 F 3 "~" H 4250 4050 50  0001 C CNN
 	1    4250 4050
@@
 F 0 "R7" V 3950 2325 50  0000 C CNN
 F 1 "1K" V 4000 2500 50  0000 C CNN
-F 2 "" V 3930 2500 50  0001 C CNN
+F 2 "Resistor_SMD:R_0805_2012Metric" V 3930 2500 50  0001 C CNN
 F 3 "~" H 4000 2500 50  0001 C CNN
 	1    4000 2500
@@
 F 0 "R2" H 1280 2554 50  0000 R CNN
 F 1 "10K" H 1280 2645 50  0000 R CNN
-F 2 "" V 1280 2600 50  0001 C CNN
+F 2 "Resistor_SMD:R_0805_2012Metric" V 1280 2600 50  0001 C CNN
 F 3 "~" H 1350 2600 50  0001 C CNN
 	1    1350 2600
@@
 F 0 "R1" H 1280 2154 50  0000 R CNN
 F 1 "100K" H 1280 2245 50  0000 R CNN
-F 2 "" V 1280 2200 50  0001 C CNN
+F 2 "Resistor_SMD:R_0805_2012Metric" V 1280 2200 50  0001 C CNN
 F 3 "~" H 1350 2200 50  0001 C CNN
 	1    1350 2200
@@
 F 0 "U2" H 7617 3147 60  0000 C CNN
 F 1 "GY-NEO6MV2" H 7617 3041 60  0000 C CNN
-F 2 "" H 7850 2700 60  0000 C CNN
+F 2 "hymTracker:Neo6" H 7850 2700 60  0000 C CNN
 F 3 "" H 7850 2700 60  0000 C CNN
 	1    7800 2750
@@
 F 0 "U1" H 3425 6525 50  0000 C CNN
 F 1 "MP1584_DCDC" H 3425 6434 50  0000 C CNN
-F 2 "" H 3450 6100 50  0001 C CNN
+F 2 "hymTracker:MP1854EN_board" H 3450 6100 50  0001 C CNN
 F 3 "" H 3450 6100 50  0001 C CNN
 	1    3450 6100
@@
 F 0 "J1" H 7818 4908 50  0000 C CNN
 F 1 "DB9_Female" H 7818 4999 50  0000 C CNN
-F 2 "" H 7900 5600 50  0001 C CNN
+F 2 "Connector_Dsub:DSUB-9_Female_Horizontal_P2.77x2.84mm_EdgePinOffset7.70mm_Housed_MountingHolesOffset9.12mm" H 7900 5600 50  0001 C CNN
 F 3 " ~" H 7900 5600 50  0001 C CNN
 	1    7900 5600

Commit message: PCD cizimi tamamlandi
Parts:
- U1: symbol mylibs:MP1584_DCDC -> hymTracker-rescue:MP1584_DCDC-mylibs
Connections:
- net labels added: VBatarya-
- wire segments 64 -> 65
Other:
- note added: "+"
- note added: "5V"
- note added: "Giris:\n3-30 Volt"
- moved on the sheet: R1, R2
Changed lines of the file:
@@
 L Device:R R2
 U 1 1 5E72518B
-P 1350 2600
-F 0 "R2" H 1280 2554 50  0000 R CNN
-F 1 "10K" H 1280 2645 50  0000 R CNN
-F 2 "Resistor_SMD:R_0805_2012Metric" V 1280 2600 50  0001 C CNN
-F 3 "~" H 1350 2600 50  0001 C CNN
-	1    1350 2600
+P 1500 3300
+F 0 "R2" H 1430 3254 50  0000 R CNN
+F 1 "10K" H 1430 3345 50  0000 R CNN
+F 2 "Resistor_SMD:R_0805_2012Metric" V 1430 3300 50  0001 C CNN
+F 3 "~" H 1500 3300 50  0001 C CNN
+	1    1500 3300
 	-1   0    0    1
 $EndComp
@@
 L Device:R R1
 U 1 1 5E72559B
-P 1350 2200
-F 0 "R1" H 1280 2154 50  0000 R CNN
-F 1 "100K" H 1280 2245 50  0000 R CNN
-F 2 "Resistor_SMD:R_0805_2012Metric" V 1280 2200 50  0001 C CNN
-F 3 "~" H 1350 2200 50  0001 C CNN
-	1    1350 2200
+P 1500 2900
+F 0 "R1" H 1430 2854 50  0000 R CNN
+F 1 "100K" H 1430 2945 50  0000 R CNN
+F 2 "Resistor_SMD:R_0805_2012Metric" V 1430 2900 50  0001 C CNN
+F 3 "~" H 1500 2900 50  0001 C CNN
+	1    1500 2900
 	-1   0    0    1
 $EndComp
@@
 L power:GND #PWR01
 U 1 1 5E72AE6E
-P 1350 2850
-F 0 "#PWR01" H 1350 2600 50  0001 C CNN
-F 1 "GND" H 1355 2677 50  0000 C CNN
-F 2 "" H 1350 2850 50  0001 C CNN
-F 3 "" H 1350 2850 50  0001 C CNN
-	1    1350 2850
-	1    0    0    -1
-$EndComp
-Wire Wire Line
-	1350 2350 1350 2400
-Wire Wire Line
-	1350 2750 1350 2850
-Connection ~ 1350 2400
-Wire Wire Line
-	1350 2400 1350 2450
-Wire Wire Line
-	1350 2400 2650 2400
+P 1500 3550
+F 0 "#PWR01" H 1500 3300 50  0001 C CNN
+F 1 "GND" H 1505 3377 50  0000 C CNN
+F 2 "" H 1500 3550 50  0001 C CNN
+F 3 "" H 1500 3550 50  0001 C CNN
+	1    1500 3550
+	1    0    0    -1
+$EndComp
+Wire Wire Line
+	1500 3450 1500 3550
 Text Label 3650 2900 0    50   ~ 0
 GPS_TXD
@@
 F 0 "U2" H 7617 3147 60  0000 C CNN
 F 1 "GY-NEO6MV2" H 7617 3041 60  0000 C CNN
-F 2 "hymTracker:Neo6" H 7850 2700 60  0000 C CNN
+F 2 "hymTracker:Neo6" H 7800 2450 60  0000 C CNN
 F 3 "" H 7850 2700 60  0000 C CNN
 	1    7800 2750
@@
 GPS_TXD
 $Comp
-L mylibs:MP1584_DCDC U1
+L hymTracker-rescue:MP1584_DCDC-mylibs U1
 U 1 1 5E700D4E
 P 3450 6100
@@
 MIKROFON
 Wire Wire Line
-	1350 2050 1350 1950
-Text Label 1350 1950 1    50   ~ 0
+	1500 2750 1500 2650
+Text Label 1500 2650 1    50   ~ 0
 Vbatarya
 Text Label 2650 2500 2    50   ~ 0
@@
 NoConn ~ 3650 2800
 NoConn ~ 2650 2700
-NoConn ~ 2650 3000
-NoConn ~ 2650 3100
 Text Label 2650 2800 2    50   ~ 0
 I2C_SDA
 Text Label 2650 2900 2    50   ~ 0
 I2C_SCL
-Wire Wire Line
-	5500 6200 5500 6400
-$Comp
-L power:GND #PWR010
-U 1 1 5E777063
-P 5500 6400
-F 0 "#PWR010" H 5500 6150 50  0001 C CNN
-F 1 "GND" H 5505 6227 50  0000 C CNN
-F 2 "" H 5500 6400 50  0001 C CNN
-F 3 "" H 5500 6400 50  0001 C CNN
-	1    5500 6400
-	1    0    0    -1
-$EndComp
+Text Label 8200 5200 0    50   ~ 0
+MIKROFON
+Text Label 8200 5400 0    50   ~ 0
+PTT
+Text Label 8200 5800 0    50   ~ 0
+I2C_SDA
 Text Label 8200 6000 0    50   ~ 0
-MIKROFON
-Text Label 8200 5800 0    50   ~ 0
-PTT
-Text Label 8200 5300 0    50   ~ 0
-I2C_SDA
-Text Label 8200 5400 0    50   ~ 0
 I2C_SCL
 Text Label 8200 5500 0    50   ~ 0
@@
 Text Label 8200 5700 0    50   ~ 0
 Vbatarya
-Text Label 3650 2100 0    50   ~ 0
+Text Label 2650 3000 2    50   ~ 0
 DIGITAL_GIRIS
 Text Label 8200 5900 0    50   ~ 0
 DIGITAL_GIRIS
-Text Label 5500 6200 1    50   ~ 0
+Text Label 4700 6300 0    50   ~ 0
 GND
-Text Label 8200 5200 0    50   ~ 0
+Text Label 8200 5300 0    50   ~ 0
 GND
+Text Notes 1900 6100 0    50   ~ 0
+Giris:\n3-30 Volt
+Text Notes 4700 6000 0    50   ~ 0
+5V
+Text Notes 2200 5900 0    50   ~ 0
++
+Wire Wire Line
+	2750 6300 2250 6300
+Text Label 2250 6300 2    50   ~ 0
+VBatarya-
+Wire Wire Line
+	4100 6300 4700 6300
+Wire Wire Line
+	1500 3050 1500 3100
+NoConn ~ 2650 2400
+Wire Wire Line
+	2650 3100 1500 3100
+Connection ~ 1500 3100
+Wire Wire Line
+	1500 3100 1500 3150
+NoConn ~ 3650 2100
 $EndSCHEMATC
