File: Hardware/hymTracker/hymTracker.kicad_pcb (KiCad board)
At the start: 2 copper layers, 45.7 x 54.6 mm, 19 parts, among them J1 DB9_Female, Q1 2N7000, U1 MP1584_DCDC, U2 GY-NEO6MV2

Commit message: PCB logo
Routing:
- net /GPS_TXD: track 38.3 -> 27.3 mm

Commit message: yeni 3d elemanlar
Other:
- board text added: "TAMSAT hymTracker"
Changed lines of the file:
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@@
   (general
     (thickness 1.6)
-    (drawings 14)
+    (drawings 16)
     (tracks 352)
     (zones 0)
@@
     (pad 1 thru_hole circle (at -16.256 2.286) (size 2.2 2.2) (drill 0.762) (layers *.Cu *.Mask)
       (net 3 /VCC))
+    (model ${KIPRJMOD}/hymTracker.pretty/gps_neo6.wrl
+      (offset (xyz -14.5 -3.5 3.5))
+      (scale (xyz 400 375 200))
+      (rotate (xyz 0 0 90))
+    )
+    (model ${KISYS3DMOD}/Connector_PinHeader_1.27mm.3dshapes/PinHeader_1x04_P1.27mm_Vertical.wrl
+      (offset (xyz -16 2.5 0))
+      (scale (xyz 1 2.1 1.5))
+      (rotate (xyz 0 0 0))
+    )
   )
   (module hymTracker:MP1854EN_board (layer F.Cu)
@@
       (effects (font (size 1 1) (thickness 0.15)))
     )
-    (fp_text value MP1584_DCDC (at 2.54 1.27) (layer F.Fab)
+    (fp_text value MP1584_DCDC (at 2.54 7.366) (layer F.Fab)
       (effects (font (size 1 1) (thickness 0.15)))
     )
@@
     (pad 1 thru_hole circle (at -7.62 -5.08 180) (size 1.524 1.524) (drill 0.762) (layers *.Cu *.Mask)
       (net 32 /Vbatarya))
+    (model "${KIPRJMOD}/hymTracker.pretty/LM2596 DC-DC Buck Converter Module.stp"
+      (offset (xyz 39 -54.5 0))
+      (scale (xyz 0.6 0.0001 0.9))
+      (rotate (xyz -90 0 0))
+    )
   )
   (module Resistor_SMD:R_0805_2012Metric (layer B.Cu)
@@
     )
   )
+  (gr_text "TAMSAT\nhymTracker" (at 89.408 51.816) (layer B.Cu)
+    (effects (font (size 1.5 1.5) (thickness 0.3)) (justify mirror))
+  )
+  (gr_text "TAMSAT\nhymTracker" (at 89.408 51.816) (layer F.Cu)
+    (effects (font (size 1.5 1.5) (thickness 0.3)))
+  )
   (dimension 54.61 (width 0.12) (layer F.SilkS)
