File: Hardware/hymTracker/hymTracker.kicad_pcb (KiCad board)
At the start: 2 copper layers, 45.7 x 54.6 mm, 19 parts, among them J1 DB9_Female, Q1 2N7000, U1 MP1584_DCDC, U2 GY-NEO6MV2

Commit message: gps ters cevrildi
Parts:
- U2: moved to F.Cu
- moved U2 2.32 mm to (81.2, 59.9)
Routing:
- net /VCC: track 31.5 -> 24.4 mm
- net GND: track 10.3 -> 5.08 mm
- net /GPS_TXD: track 27.3 -> 24.1 mm
- net /GPS_RXD: track 29.0 -> 30.8 mm
Changed lines of the file:
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@@
     (thickness 1.6)
     (drawings 22)
-    (tracks 361)
+    (tracks 357)
     (zones 0)
     (modules 19)
@@
     (solder_mask_min_width 0.25)
     (aux_axis_origin 0 0)
-    (visible_elements FFFFF77F)
+    (visible_elements FFFFFF7F)
     (pcbplotparams
       (layerselection 0x010fc_ffffffff)
@@
     )
   )
-  (module hymTracker:Neo6 (layer B.Cu)
-    (at 81.28 62.23)
-    (fp_text reference U2 (at 0.508 -0.5) (layer B.SilkS)
-      (effects (font (size 1 1) (thickness 0.15)) (justify mirror))
-    )
-    (fp_text value GY-NEO6MV2 (at 0.508 0.5) (layer B.Fab)
-      (effects (font (size 1 1) (thickness 0.15)) (justify mirror))
-    )
-    (fp_circle (center -14.986 8.89) (end -13.462 8.89) (layer B.SilkS) (width 0.12))
-    (fp_circle (center -14.986 -11.176) (end -13.462 -11.176) (layer B.SilkS) (width 0.12))
-    (fp_circle (center 14.732 -11.176) (end 16.256 -11.176) (layer B.SilkS) (width 0.12))
-    (fp_circle (center 14.732 8.89) (end 16.256 8.89) (layer B.SilkS) (width 0.12))
-    (fp_line (start -17.78 -14.224) (end -18.034 -14.224) (layer B.SilkS) (width 0.12))
-    (fp_line (start -18.034 -14.224) (end -18.034 11.938) (layer B.SilkS) (width 0.12))
-    (fp_line (start 17.78 -14.224) (end -17.78 -14.224) (layer B.SilkS) (width 0.12))
-    (fp_line (start 17.78 11.938) (end 17.78 -14.224) (layer B.SilkS) (width 0.12))
-    (fp_line (start -18.034 11.938) (end 17.78 11.938) (layer B.SilkS) (width 0.12))
-    (pad 4 thru_hole circle (at -16.256 -5.334) (size 2.2 2.2) (drill 0.762) (layers *.Cu *.Mask)
-      (net 5 GND))
-    (pad 3 thru_hole circle (at -16.256 -2.794) (size 2.2 2.2) (drill 0.762) (layers *.Cu *.Mask)
+  (module hymTracker:Neo6 (layer F.Cu)
+    (at 81.25 59.91)
+    (fp_text reference U2 (at 0.508 0.5) (layer F.SilkS)
+      (effects (font (size 1 1) (thickness 0.15)))
+    )
+    (fp_text value GY-NEO6MV2 (at 0.508 -0.5) (layer F.Fab)
+      (effects (font (size 1 1) (thickness 0.15)))
+    )
+    (fp_circle (center -14.986 -8.89) (end -13.462 -8.89) (layer F.SilkS) (width 0.12))
+    (fp_circle (center -14.986 11.176) (end -13.462 11.176) (layer F.SilkS) (width 0.12))
+    (fp_circle (center 14.732 11.176) (end 16.256 11.176) (layer F.SilkS) (width 0.12))
+    (fp_circle (center 14.732 -8.89) (end 16.256 -8.89) (layer F.SilkS) (width 0.12))
+    (fp_line (start -17.78 14.224) (end -18.034 14.224) (layer F.SilkS) (width 0.12))
+    (fp_line (start -18.034 14.224) (end -18.034 -11.938) (layer F.SilkS) (width 0.12))
+    (fp_line (start 17.78 14.224) (end -17.78 14.224) (layer F.SilkS) (width 0.12))
+    (fp_line (start 17.78 -11.938) (end 17.78 14.224) (layer F.SilkS) (width 0.12))
+    (fp_line (start -18.034 -11.938) (end 17.78 -11.938) (layer F.SilkS) (width 0.12))
+    (pad 4 thru_hole circle (at -16.256 5.334) (size 2.2 2.2) (drill 0.762) (layers *.Cu *.Mask)
+      (net 5 GND))
+    (pad 3 thru_hole circle (at -16.256 2.794) (size 2.2 2.2) (drill 0.762) (layers *.Cu *.Mask)
       (net 4 /GPS_TXD))
-    (pad 2 thru_hole circle (at -16.256 -0.254) (size 2.2 2.2) (drill 0.762) (layers *.Cu *.Mask)
+    (pad 2 thru_hole circle (at -16.256 0.254) (size 2.2 2.2) (drill 0.762) (layers *.Cu *.Mask)
       (net 2 /GPS_RXD))
-    (pad 1 thru_hole circle (at -16.256 2.286) (size 2.2 2.2) (drill 0.762) (layers *.Cu *.Mask)
+    (pad 1 thru_hole circle (at -16.256 -2.286) (size 2.2 2.2) (drill 0.762) (layers *.Cu *.Mask)
       (net 3 /VCC))
     (model ${KISYS3DMOD}/Connector_PinHeader_1.27mm.3dshapes/PinHeader_1x04_P1.27mm_Vertical.wrl
@@
   (segment (start 84.1525 77.1375) (end 83.82 77.47) (width 0.4) (layer B.Cu) (net 1))
   (segment (start 84.1525 74.93) (end 84.1525 77.1375) (width 0.4) (layer B.Cu) (net 1))
-  (segment (start 67.056 64.008) (end 67.056 66.04) (width 0.4) (layer F.Cu) (net 2))
+  (segment (start 61.759999 86.830001) (end 60.96 87.63) (width 0.4) (layer F.Cu) (net 2))
+  (segment (start 66.96 62.13) (end 66.96 66.136) (width 0.4) (layer F.Cu) (net 2))
+  (segment (start 64.994 60.164) (end 66.96 62.13) (width 0.4) (layer F.Cu) (net 2))
+  (segment (start 63.59201 84.99799) (end 61.759999 86.830001) (width 0.4) (layer F.Cu) (net 2))
+  (segment (start 66.96 66.136) (end 63.59201 69.50399) (width 0.4) (layer F.Cu) (net 2))
   (segment (start 63.59201 69.50399) (end 63.59201 84.99799) (width 0.4) (layer F.Cu) (net 2))
-  (segment (start 65.024 61.976) (end 67.056 64.008) (width 0.4) (layer F.Cu) (net 2))
-  (segment (start 63.59201 84.99799) (end 61.759999 86.830001) (width 0.4) (layer F.Cu) (net 2))
-  (segment (start 61.759999 86.830001) (end 60.96 87.63) (width 0.4) (layer F.Cu) (net 2))
-  (segment (start 67.056 66.04) (end 63.59201 69.50399) (width 0.4) (layer F.Cu) (net 2))
   (segment (start 80.518 57.15) (end 80.518 59.69) (width 0.4) (layer B.Cu) (net 3))
   (segment (start 76.2 52.07) (end 78.74 52.07) (width 0.8) (layer F.Cu) (net 3))
   (segment (start 80.518 53.848) (end 80.518 57.15) (width 0.8) (layer F.Cu) (net 3))
   (segment (start 78.74 52.07) (end 80.518 53.848) (width 0.8) (layer F.Cu) (net 3))
-  (segment (start 72.644 62.992) (end 66.548 62.992) (width 0.4) (layer B.Cu) (net 3))
-  (segment (start 66.548 62.992) (end 65.024 64.516) (width 0.4) (layer B.Cu) (net 3))
-  (segment (start 74.676 60.96) (end 72.644 62.992) (width 0.4) (layer B.Cu) (net 3))
   (segment (start 76.2 52.07) (end 74.676 53.594) (width 0.4) (layer B.Cu) (net 3))
-  (segment (start 74.676 53.594) (end 74.676 60.96) (width 0.4) (layer B.Cu) (net 3))
+  (segment (start 69.024 53.594) (end 64.994 57.624) (width 0.4) (layer B.Cu) (net 3))
+  (segment (start 74.676 53.594) (end 69.024 53.594) (width 0.4) (layer B.Cu) (net 3))
+  (segment (start 64.994 62.704) (end 62.992 64.706) (width 0.4) (layer F.Cu) (net 4))
   (segment (start 62.992 83.058) (end 60.96 85.09) (width 0.4) (layer F.Cu) (net 4))
-  (segment (start 65.024 59.436) (end 62.992 61.468) (width 0.4) (layer F.Cu) (net 4))
-  (segment (start 62.992 61.468) (end 62.992 83.058) (width 0.4) (layer F.Cu) (net 4))
+  (segment (start 62.992 64.706) (end 62.992 83.058) (width 0.4) (layer F.Cu) (net 4))
   (via (at 101.6 45.72) (size 0.8) (drill 0.4) (layers F.Cu B.Cu) (net 5))
   (via (at 101.6 92.71) (size 0.8) (drill 0.4) (layers F.Cu B.Cu) (net 5))
@@
   (via (at 60.96 43.18) (size 0.8) (drill 0.4) (layers F.Cu B.Cu) (net 5))
   (via (at 99.06 43.18) (size 0.8) (drill 0.4) (layers F.Cu B.Cu) (net 5))
-  (segment (start 62.23 59.69) (end 65.024 56.896) (width 0.4) (layer F.Cu) (net 5))
-  (segment (start 60.96 59.69) (end 62.23 59.69) (width 0.4) (layer F.Cu) (net 5))
   (segment (start 99.06 46.482) (end 99.06 49.022) (width 0.4) (layer B.Cu) (net 5))
   (segment (start 80.518 46.482) (end 80.518 49.022) (width 0.4) (layer B.Cu) (net 5))

Commit message: dual version
Other:
- board text added: "TA7W"
Changed lines of the file:
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@@
   (general
     (thickness 1.6)
-    (drawings 22)
+    (drawings 23)
     (tracks 357)
     (zones 0)
@@
     )
   )
+  (gr_text TA7W (at 69.5 81.27 90) (layer F.Cu)
+    (effects (font (size 1.7 1.7) (thickness 0.3)))
+  )
   (gr_text "hymTR\niZCi" (at 67.28 91.47) (layer B.Cu)
